Commit message: ..

File: viberobotics/assets/urdf/SundayA1_full_2dof_arm/robot.urdf (robot description, URDF)
Before this commit: robot SundayA1_URDF, 13 links, 12 joints
Links:
- removed link sole0120
- removed link sole0120mir
- added link elbow, mass 0.0815874; collision mesh filename=assets/elbow1216.stl; collision mesh filename=assets/sts3215.stl
- added link elbow_2, mass 0.0815874; collision mesh filename=assets/elbow1216.stl; collision mesh filename=assets/sts3215.stl
- added link head1209, mass 1e-09; collision mesh filename=assets/head1209.stl; collision mesh filename=assets/max4466.stl
- added link left_foot0120, mass 0.0592492; collision mesh filename=assets/left_foot0120.stl; visual mesh filename=assets/left_foot0120.stl
- added link left_hand, mass 0.0947896; collision mesh filename=assets/left_paw0123.stl; collision mesh filename=assets/sts3215.stl
- added link right_foot0120, mass 0.0592497; collision mesh filename=assets/right_foot0120.stl; visual mesh filename=assets/right_foot0120.stl
- added link right_hand, mass 0.0947896; collision mesh filename=assets/right_paw0123.stl; collision mesh filename=assets/sts3215.stl
- added link right_wrist0124, mass 0.149125; collision mesh filename=assets/right_wrist0124.stl; collision mesh filename=assets/sts3215.stl
- added link shoulder, mass 0.0228612; collision mesh filename=assets/shoulder0124.stl; visual mesh filename=assets/shoulder0124.stl
- added link shoulder_2, mass 0.0228612; collision mesh filename=assets/shoulder0124.stl; visual mesh filename=assets/shoulder0124.stl
- added link sts3215_3, mass 0.146992; collision mesh filename=assets/left_ankle0120.stl; collision mesh filename=assets/sts3215.stl
- added link thumb_0112, mass 0.0051587; collision mesh filename=assets/thumb_0112.stl; visual mesh filename=assets/thumb_0112.stl
- added link thumb_0112_2, mass 0.0051587; collision mesh filename=assets/thumb_0112.stl; visual mesh filename=assets/thumb_0112.stl
- link body: mass 0.460845 -> 1.01051; geometry collision mesh filename=assets/internal_weight_395g__configuration_default.stl; collision mesh filename=assets/leg_foundation1029.stl
- link hip: geometry collision mesh filename=assets/hips1016.stl; collision mesh filename=assets/sts3215.stl
- link hip_2: geometry collision mesh filename=assets/hips1016.stl; collision mesh filename=assets/sts3215.stl
- link knee: geometry collision mesh filename=assets/calf1016.stl; collision mesh filename=assets/sts3215.stl
- link knee_2: geometry collision mesh filename=assets/calf1016.stl; collision mesh filename=assets/sts3215.stl
- link knee_down: geometry collision mesh filename=assets/knee_down.stl; visual mesh filename=assets/knee_down.stl
- link knee_down_2: geometry collision mesh filename=assets/knee_down.stl; visual mesh filename=assets/knee_down.stl
- link low_hip: mass 0.0781435 -> 0.0839507; geometry collision mesh filename=assets/sts3215.stl; collision mesh filename=assets/thigh1111.stl
- link low_hip_2: mass 0.0781435 -> 0.0839507; geometry collision mesh filename=assets/sts3215.stl; collision mesh filename=assets/thigh1111.stl
- link sts3215: geometry collision mesh filename=assets/right_ankle0120.stl; collision mesh filename=assets/sts3215.stl
- link sts3215_2: mass 0.146992 -> 0.149125; geometry collision mesh filename=assets/left_wrist0124.stl; collision mesh filename=assets/sts3215.stl
Joints:
- added joint head_yaw: type revolute, parent body, child head1209, origin xyz=4.68418e-10 0.018593 0.206868 rpy=-3.14159 -3.1481e-28 -3.14159, axis 0 0 1, limit lower=-1 upper=1 effort=1.9 velocity=5
- added joint left_elbow_pitch: type revolute, parent elbow_2, child sts3215_2, origin xyz=0.018825 -0.080054 -0.01905 rpy=-2.34193e-31 1.5708 0, axis 0 0 1, limit lower=-3.141592653589793 upper=3.141592653589793 effort=1.9 velocity=5
- added joint left_hand: type revolute, parent left_hand, child thumb_0112_2, origin xyz=0.01905 -0.0125 -0.028 rpy=1.92819e-09 -1.5708 0, axis 0 0 1, limit lower=0 upper=2.5 effort=1.9 velocity=5
- added joint left_shoulder_pitch: type revolute, parent body, child shoulder_2, origin xyz=-0.0905929 0.019393 0.173135 rpy=-1.5708 4.20136e-17 -1.5708, axis 0 0 1, limit lower=-0.785 upper=0.785 effort=1.9 velocity=5
- added joint left_shoulder_roll: type revolute, parent shoulder_2, child elbow_2, origin xyz=-0.019 -2.77556e-17 -0.049 rpy=3.14159 1.5708 0, axis 0 0 1, limit lower=-1.7 upper=1.7 effort=1.9 velocity=5
- added joint left_wrist_yaw: type revolute, parent sts3215_2, child left_hand, origin xyz=-5.4e-05 -0.085209 -0.01905 rpy=-1.5708 -1.5708 0, axis 0 0 1, limit lower=-3.141592653589793 upper=3.141592653589793 effort=1.9 velocity=5
- added joint right_elbow_pitch: type revolute, parent elbow, child right_wrist0124, origin xyz=-0.018825 -0.080054 -0.01905 rpy=-1.68325e-15 -1.5708 0, axis 0 0 1, limit lower=-3.141592653589793 upper=3.141592653589793 effort=1.9 velocity=5
- added joint right_hand: type revolute, parent right_hand, child thumb_0112, origin xyz=-0.01905 -0.012554 -0.028 rpy=-3.14159 1.5708 0, axis 0 0 1, limit lower=-2.5 upper=0 effort=1.9 velocity=5
- added joint right_shoulder_pitch: type revolute, parent body, child shoulder, origin xyz=0.0905929 0.019393 0.169381 rpy=1.5708 -1.92775e-17 1.5708, axis 0 0 1, limit lower=-0.785 upper=0.785 effort=1.9 velocity=5
- added joint right_shoulder_roll: type revolute, parent shoulder, child elbow, origin xyz=0.019 1.11022e-16 0.049 rpy=-9.24412e-16 1.5708 0, axis 0 0 1, limit lower=-1.7 upper=1.7 effort=1.9 velocity=5
- added joint right_wrist_yaw: type revolute, parent right_wrist0124, child right_hand, origin xyz=-7.28584e-17 -0.085209 -0.01905 rpy=-1.5708 1.5708 0, axis 0 0 1, limit lower=-3.141592653589793 upper=3.141592653589793 effort=1.9 velocity=5
- joint left_ankle_pitch: child sts3215_2 -> sts3215_3; origin xyz=-2.01228e-16 -0.05 -0.000225009 rpy=-6.21725e-15 -9.99201e-16 1.02085e-14 -> xyz=1.49186e-16 -0.0500539 -0.000225009 rpy=-6.21725e-15 2.94918e-15 1.02085e-14
- joint left_ankle_roll: child sole0120 -> left_foot0120; origin xyz=0.03295 -0.024834 -0.01905 rpy=-3.14159 -1.5708 0 -> xyz=0.03295 -0.024834 -0.01905 rpy=-2.77556e-16 1.5708 0; parent sts3215_2 -> sts3215_3
- joint left_hip_roll: origin xyz=-0.0617138 0.0538513 0.0336753 rpy=2.26893 3.60356e-15 1.5708 -> xyz=-0.067812 0.019393 -0.0153431 rpy=2.26893 3.60356e-15 1.5708
- joint left_knee: origin xyz=6.93889e-18 -0.019 -0.059 rpy=1.5708 6.03027e-14 -3.00469e-15 -> xyz=1.04083e-17 -0.019 -0.059 rpy=1.5708 6.03027e-14 -3.00469e-15
- joint right_ankle_pitch: origin xyz=-1.38778e-17 0.05 0.000225009 rpy=3.14159 -2.9663e-16 5.92467e-14 -> xyz=2.70617e-16 0.0500539 0.000225009 rpy=-3.14159 -1.11022e-16 7.57221e-14
- joint right_ankle_roll: child sole0120mir -> right_foot0120; origin xyz=-0.03295 -0.024834 -0.01905 rpy=4.03525e-30 -1.5708 0 -> xyz=-0.03295 -0.024888 -0.01905 rpy=-1.5708 1.54565 1.5708
- joint right_hip_pitch: origin xyz=0.01905 -0.05 0.018825 rpy=-1.5708 0.698132 1.5708 -> xyz=0.01905 -0.05 0.018825 rpy=-1.5708 0.67299 1.5708
- joint right_hip_roll: origin xyz=0.0618745 0.0538513 0.0334838 rpy=2.26893 -7.32543e-14 -1.5708 -> xyz=0.0679727 0.019393 -0.0155346 rpy=2.26893 -7.32817e-14 -1.5708
- joint right_hip_yaw: origin xyz=-0.02695 -6.80012e-16 0.018825 rpy=-7.77156e-16 1.5708 0 -> xyz=-0.02695 -6.10623e-16 0.018825 rpy=1.95974e-15 1.5708 0
- joint right_knee: origin xyz=4.16334e-17 0.019 -0.059 rpy=-1.5708 -7.00545e-14 -3.14159 -> xyz=1.38778e-17 0.019 -0.059 rpy=-1.5708 -5.73863e-14 -3.14159
